File: pcb/PlantMonitor/PlantMonitor.brd (EAGLE design)
At the start: 108 x 29 mm, 28 parts, among them IC1 453-00005

Commit message: Code adoptation for new board - low battery detection - reading ID and sensitivity keys using 2 analogue inputs - improved status indication
Parts:
- R10, R6: value 40k -> 39k
- R11, R7: value 80k -> 82k
- R12: value 5k -> 6.8k
- R2: value 820 -> 390
- R3: value 2.2k -> 4.7k
- R5, R9: value 20k -> 22k
Changed lines of the file:
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@@
 <layers>
 <layer number="1" name="Top" color="4" fill="1" visible="yes" active="yes"/>
-<layer number="16" name="Bottom" color="1" fill="1" visible="no" active="yes"/>
+<layer number="16" name="Bottom" color="1" fill="1" visible="yes" active="yes"/>
 <layer number="17" name="Pads" color="2" fill="1" visible="yes" active="yes"/>
 <layer number="18" name="Vias" color="2" fill="1" visible="yes" active="yes"/>
@@
 <attribute name="RS_PRICE-STOCK" value="" x="5.715" y="13.97" size="1.778" layer="27" rot="R90" display="off"/>
 </element>
-<element name="R3" library="rcl" library_urn="urn:adsk.eagle:library:334" package="R0603" package3d_urn="urn:adsk.eagle:package:23555/2" value="2.2k" x="12.7" y="5.715" smashed="yes" rot="R180">
+<element name="R3" library="rcl" library_urn="urn:adsk.eagle:library:334" package="R0603" package3d_urn="urn:adsk.eagle:package:23555/2" value="4.7k" x="12.7" y="5.715" smashed="yes" rot="R180">
 <attribute name="NAME" x="13.335" y="7.366" size="0.762" layer="25" rot="R180"/>
 <attribute name="VALUE" x="13.335" y="7.62" size="1.27" layer="27" rot="R180"/>
@@
 <attribute name="VALUE" x="13.335" y="3.81" size="1.27" layer="27" rot="R180"/>
 </element>
-<element name="R2" library="rcl" library_urn="urn:adsk.eagle:library:334" package="R0603" package3d_urn="urn:adsk.eagle:package:23555/2" value="820" x="12.7" y="3.81" smashed="yes" rot="R180">
+<element name="R2" library="rcl" library_urn="urn:adsk.eagle:library:334" package="R0603" package3d_urn="urn:adsk.eagle:package:23555/2" value="390" x="12.7" y="3.81" smashed="yes" rot="R180">
 <attribute name="NAME" x="11.049" y="4.191" size="0.762" layer="25" rot="R180"/>
 <attribute name="VALUE" x="13.335" y="5.715" size="1.27" layer="27" rot="R180"/>
@@
 <element name="U$2" library="STLib" package="COIN-CELL-HOLDER" value="COIN-CELL-HOLDER" x="9.525" y="13.335" rot="MR270"/>
 <element name="U$3" library="STLib" package="MICRO-BUZZER" value="MICRO-BUZZER" x="23.18" y="21.19" rot="MR180"/>
-<element name="R12" library="rcl" library_urn="urn:adsk.eagle:library:334" package="R0603" package3d_urn="urn:adsk.eagle:package:23555/2" value="5k" x="23.495" y="3.81" smashed="yes">
+<element name="R12" library="rcl" library_urn="urn:adsk.eagle:library:334" package="R0603" package3d_urn="urn:adsk.eagle:package:23555/2" value="6.8k" x="23.495" y="3.81" smashed="yes">
 <attribute name="NAME" x="22.606" y="4.699" size="0.762" layer="25"/>
 <attribute name="VALUE" x="22.86" y="1.905" size="1.27" layer="27"/>
@@
 <attribute name="VALUE" x="27.432" y="9.2075" size="1.27" layer="27" rot="R180"/>
 </element>
-<element name="R5" library="rcl" library_urn="urn:adsk.eagle:library:334" package="R0603" package3d_urn="urn:adsk.eagle:package:23555/2" value="20k" x="26.797" y="8.5725" smashed="yes" rot="R180">
+<element name="R5" library="rcl" library_urn="urn:adsk.eagle:library:334" package="R0603" package3d_urn="urn:adsk.eagle:package:23555/2" value="22k" x="26.797" y="8.5725" smashed="yes" rot="R180">
 <attribute name="NAME" x="27.36" y="4.4075" size="0.762" layer="25" rot="R180"/>
 <attribute name="VALUE" x="27.432" y="10.4775" size="1.27" layer="27" rot="R180"/>
 </element>
-<element name="R6" library="rcl" library_urn="urn:adsk.eagle:library:334" package="R0603" package3d_urn="urn:adsk.eagle:package:23555/2" value="40k" x="26.797" y="9.8425" smashed="yes" rot="R180">
+<element name="R6" library="rcl" library_urn="urn:adsk.eagle:library:334" package="R0603" package3d_urn="urn:adsk.eagle:package:23555/2" value="39k" x="26.797" y="9.8425" smashed="yes" rot="R180">
 <attribute name="NAME" x="27.36" y="5.3775" size="0.762" layer="25" rot="R180"/>
 <attribute name="VALUE" x="27.432" y="11.7475" size="1.27" layer="27" rot="R180"/>
 </element>
-<element name="R7" library="rcl" library_urn="urn:adsk.eagle:library:334" package="R0603" package3d_urn="urn:adsk.eagle:package:23555/2" value="80k" x="26.797" y="11.1125" smashed="yes" rot="R180">
+<element name="R7" library="rcl" library_urn="urn:adsk.eagle:library:334" package="R0603" package3d_urn="urn:adsk.eagle:package:23555/2" value="82k" x="26.797" y="11.1125" smashed="yes" rot="R180">
 <attribute name="NAME" x="27.36" y="6.3475" size="0.762" layer="25" rot="R180"/>
 <attribute name="VALUE" x="27.432" y="13.0175" size="1.27" layer="27" rot="R180"/>
@@
 <attribute name="VALUE" x="27.432" y="14.2875" size="1.27" layer="27" rot="R180"/>
 </element>
-<element name="R9" library="rcl" library_urn="urn:adsk.eagle:library:334" package="R0603" package3d_urn="urn:adsk.eagle:package:23555/2" value="20k" x="26.797" y="13.6525" smashed="yes" rot="R180">
+<element name="R9" library="rcl" library_urn="urn:adsk.eagle:library:334" package="R0603" package3d_urn="urn:adsk.eagle:package:23555/2" value="22k" x="26.797" y="13.6525" smashed="yes" rot="R180">
 <attribute name="NAME" x="27.56" y="18.8875" size="0.762" layer="25" rot="R180"/>
 <attribute name="VALUE" x="27.432" y="15.5575" size="1.27" layer="27" rot="R180"/>
 </element>
-<element name="R10" library="rcl" library_urn="urn:adsk.eagle:library:334" package="R0603" package3d_urn="urn:adsk.eagle:package:23555/2" value="40k" x="26.797" y="14.9225" smashed="yes" rot="R180">
+<element name="R10" library="rcl" library_urn="urn:adsk.eagle:library:334" package="R0603" package3d_urn="urn:adsk.eagle:package:23555/2" value="39k" x="26.797" y="14.9225" smashed="yes" rot="R180">
 <attribute name="NAME" x="28.168" y="19.8575" size="0.762" layer="25" rot="R180"/>
 <attribute name="VALUE" x="27.432" y="16.8275" size="1.27" layer="27" rot="R180"/>
 </element>
-<element name="R11" library="rcl" library_urn="urn:adsk.eagle:library:334" package="R0603" package3d_urn="urn:adsk.eagle:package:23555/2" value="80k" x="26.797" y="16.1925" smashed="yes" rot="R180">
+<element name="R11" library="rcl" library_urn="urn:adsk.eagle:library:334" package="R0603" package3d_urn="urn:adsk.eagle:package:23555/2" value="82k" x="26.797" y="16.1925" smashed="yes" rot="R180">
 <attribute name="NAME" x="28.168" y="20.8275" size="0.762" layer="25" rot="R180"/>
 <attribute name="VALUE" x="27.432" y="18.0975" size="1.27" layer="27" rot="R180"/>
